File: LED-Matrix-schematic.kicad_sch (KiCad schematic)
At the start: 66 parts, among them J1 Conn_02x07_Odd_Even_MountingP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, M201 74HC595

Commit message: add filter cap
Parts:
- added C1: C, symbol Device:C
Connections:
- net at J1.5 (Pin_5), M201.10 (~{SRCLR}), M201.16 (VCC): now also C1.2
- net at J1.6 (Pin_6), J1.7 (Pin_7), M201.8 (GND): now also C1.1
Changed lines of the file:
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@@
 	)
 	(junction
+		(at 73.66 138.43)
+		(diameter 0)
+		(color 0 0 0 0)
+	)
+	(junction
 		(at 135.89 67.31)
 		(diameter 0)
@@
 	)
 	(junction
+		(at 76.2 129.54)
+		(diameter 0)
+		(color 0 0 0 0)
+	)
+	(junction
 		(at 132.08 90.17)
 		(diameter 0)
@@
 	(wire
 		(pts
+			(xy 73.66 114.3) (xy 73.66 138.43)
+		)
+		(stroke
+			(width 0)
+			(type default)
+		)
+	)
+	(wire
+		(pts
 			(xy 144.78 90.17) (xy 148.59 90.17)
 		)
@@
 	(wire
 		(pts
-			(xy 73.66 143.51) (xy 73.66 114.3)
+			(xy 73.66 143.51) (xy 73.66 138.43)
 		)
 		(stroke
@@
 	(wire
 		(pts
+			(xy 76.2 129.54) (xy 76.2 167.64)
+		)
+		(stroke
+			(width 0)
+			(type default)
+		)
+	)
+	(wire
+		(pts
 			(xy 170.18 80.01) (xy 173.99 80.01)
 		)
@@
 	(wire
 		(pts
-			(xy 76.2 123.19) (xy 76.2 167.64)
+			(xy 76.2 123.19) (xy 76.2 129.54)
 		)
 		(stroke
@@
 	(wire
 		(pts
+			(xy 64.77 129.54) (xy 76.2 129.54)
+		)
+		(stroke
+			(width 0)
+			(type default)
+		)
+	)
+	(wire
+		(pts
 			(xy 132.08 100.33) (xy 135.89 100.33)
 		)
@@
 	(wire
 		(pts
+			(xy 64.77 129.54) (xy 64.77 130.81)
+		)
+		(stroke
+			(width 0)
+			(type default)
+		)
+	)
+	(wire
+		(pts
 			(xy 52.07 165.1) (xy 121.92 165.1)
 		)
@@
 	(wire
 		(pts
+			(xy 73.66 138.43) (xy 64.77 138.43)
+		)
+		(stroke
+			(width 0)
+			(type default)
+		)
+	)
+	(wire
+		(pts
 			(xy 121.92 165.1) (xy 121.92 153.67)
 		)
@@
 					(unit 1)
 				)
+			)
+		)
+	)
+	(symbol
+		(lib_id "Device:C")
+		(at 64.77 134.62 0)
+		(unit 1)
+		(exclude_from_sim no)
+		(in_bom yes)
+		(on_board yes)
+		(dnp no)
+		(fields_autoplaced yes)
+		(property "Reference" "C1"
+			(at 68.58 133.3499 0)
+			(effects
+				(font
+					(size 1.27 1.27)
+				)
+				(justify left)
+			)
+		)
+		(property "Value" "C"
+			(at 68.58 135.8899 0)
+			(effects
+				(font
+					(size 1.27 1.27)
+				)
+				(justify left)
+			)
+		)
+		(property "Footprint" ""
+			(at 65.7352 138.43 0)
+			(effects
+				(font
+					(size 1.27 1.27)
+				)
+				(hide yes)
+			)
+		)
+		(property "Datasheet" "~"
+			(at 64.77 134.62 0)
+			(effects
+				(font
+					(size 1.27 1.27)
+				)
+				(hide yes)
+			)
+		)
+		(property "Description" "Unpolarized capacitor"
+			(at 64.77 134.62 0)
+			(effects
+				(font
+					(size 1.27 1.27)
+				)
+				(hide yes)
+			)
+		)
+		(pin "2"
+		)
+		(pin "1"
+		)
+		(instances
+			(project ""
+				(path "/86beab3a-0cbe-4d3f-ad47-35e01ac008a0"
+					(reference "C1")
+					(unit 1)
+				)
